File: TinyPICO/Shield_INA219.brd (EAGLE design)
At the start: 31.9 x 17.8 mm, 11 parts, among them J1 3.5mm, U1 INA219BIDCNT

Commit message: Prettied up the boards a little
Parts:
- added R5+, R5-: (no value), wirepad:1,6/0,9
- moved R6 2.50 mm to (20.8, 7.92)
- moved A0 2.50 mm to (15.3, 12.7)
- moved A1 2.50 mm to (17.8, 12.7)
- moved C1 2.50 mm to (20.3, 12.5)
- moved R5 2.50 mm to (11.9, 8.89)
- moved U1 2.50 mm to (16.6, 8.23)
- moved J1 0.65 mm to (3.68, 8.89)
- moved JP2 0.65 mm to (4.95, 14.0)
Connections:
- net VIN1+: now also R5+.1
- net VIN1-: now also R5-.1
Routing:
- net GND: track 6.06 -> 21.7 mm
- net VIN1+: track 17.6 -> 21.8 mm, vias 1 -> 0
- net VIN1-: track 22.1 -> 25.9 mm, vias 1 -> 0
- net 3.3V: track 28.6 -> 31.6 mm
- net SCL: track 12.1 -> 14.8 mm
- net SDA: track 8.98 -> 10.6 mm
Other:
- board text added: "INA219 SHIELD v1"
- board text removed: "INA219 SHIELD"
