File: Adafruit/INA219x2 FeatherWing.brd (EAGLE design)
At the start: 50.8 x 22.9 mm, 29 parts, among them J1 3.5mm, J2 3.5mm, U1 INA219BIDCNT, U2 INA219BIDCNT

Commit message: INA219 FeatherWing v2
Parts:
- removed JP1: (no value), microbuilder:1X12_ROUND_76MIL
- removed JP2: (no value), microbuilder:1X02_ROUND
- removed R5: 0.1/1% (PT2512FK-070R1L), microbuilder:2512
- removed R5+, R5-: (no value), wirepad:1,6/0,9
- removed R6: 10K, microbuilder:RESPACK_4X0603
- added R3: 0.1/1% (PT2512FK-070R1L), microbuilder:2512
- added R3+, R3-: (no value), wirepad:1,6/0,9
- added R4: 10K, microbuilder:RESPACK_4X0603
- JP3: device microbuilder:1X16_ROUND_76MIL -> microbuilder:1X02_ROUND
- moved R1+ 33.7 mm to (41.7, 6.60)
- moved R1- 33.6 mm to (41.7, 16.3)
- moved R1 32.3 mm to (41.7, 11.4), turned to 270 degrees
- moved JP3 20.5 mm to (45.7, 6.35), turned to 0 degrees
- moved R2 14.2 mm to (32.6, 12.4), turned to 90 degrees
Connections:
- removed net A: JP3.12, MS1.5
- removed net AREF: JP3.14, MS1.3
- removed net B: JP3.11, MS1.6
- removed net C: JP3.10, MS1.7
- removed net D: JP3.9, MS1.8
- removed net E: JP3.8, MS1.9
- removed net EN: JP1.2, MS1.27
- removed net F: JP3.7, MS1.10
- removed net G: JP3.1, MS1.16
- removed net H: JP1.10, MS1.19
- removed net I: JP1.9, MS1.20
- removed net J: JP1.8, MS1.21
- removed net K: JP1.7, MS1.22
- removed net L: JP1.6, MS1.23
- removed net M: JP1.5, MS1.24
- removed net MISO: JP3.4, MS1.13
- removed net MOSI: JP3.5, MS1.12
- removed net N: JP1.4, MS1.25
- removed net RESET: JP3.16, MS1.1
- removed net RX: JP3.3, MS1.14
- removed net SCK: JP3.6, MS1.11
- removed net TX: JP3.2, MS1.15
- removed net USB: JP1.3, MS1.26
- removed net VBAT: JP1.1, MS1.28
- net 3.3V: now also R4.5, R4.6; no longer JP3.15, R6.5, R6.6
- net GND: now also R4.7, R4.8; no longer JP3.13, R6.7, R6.8
- net N$1: now also R2.1; no longer R6.1
- net N$2: now also R2.2; no longer R6.2
- net N$3: now also R4.1; no longer R2.1
- net N$4: now also R4.2; no longer R2.2
- net SCL: now also R4.3; no longer JP1.11, R6.3
- net SDA: now also R4.4; no longer JP1.12, R6.4
- net VIN1+: now also JP3.2, R1+.1, R1.2; no longer JP2.2, R5+.1, R5.2
- net VIN1-: now also JP3.1, R1-.1, R1.1; no longer JP2.1, R5-.1, R5.1
- net VIN2+: now also R3+.1, R3.2; no longer R1+.1, R1.2
- net VIN2-: now also R3-.1, R3.1; no longer R1-.1, R1.1
Routing:
- net GND: track 26.7 -> 30.4 mm
- net VBAT: track 2.58 -> 0.00 mm
- net N: track 2.58 -> 0.00 mm
- net M: track 2.58 -> 0.00 mm
- net J: track 2.58 -> 0.00 mm
- net H: track 2.58 -> 0.00 mm
- net USB: track 2.58 -> 0.00 mm
- net L: track 2.58 -> 0.00 mm
- net K: track 2.58 -> 0.00 mm
- net EN: track 2.58 -> 0.00 mm
- net I: track 2.58 -> 0.00 mm
- net RX: track 2.56 -> 0.00 mm
- net MOSI: track 2.56 -> 0.00 mm
- net E: track 2.56 -> 0.00 mm
- net D: track 2.56 -> 0.00 mm
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Other:
- board text added: "INA219 x 2 FeatherWing v2"
- board text removed: "INA219x2 FWing v1"
- board text removed: "mi"
- board text removed: "mo"
- board text removed: "rx"
- board text removed: "sck"
- board text removed: "tx"
