File: Adafruit/INA219x2 FeatherWing.sch (EAGLE design)
At the start: 23 parts, among them J1 3.5mm, J2 3.5mm, U1 INA219BIDCNT, U2 INA219BIDCNT

Commit message: INA219 FeatherWing v2
Parts:
- removed JP1: (no value), microbuilder:HEADER-1X1276MIL
- removed JP2: (no value), microbuilder:HEADER-1X2ROUND
- removed R5: 0.1/1% (PT2512FK-070R1L), microbuilder:RESISTOR2512
- removed R5+, R5-: (no value), wirepad:1,6/0,9
- removed R6: 10K, microbuilder:RESISTOR_4PACK
- added R3: 0.1/1% (PT2512FK-070R1L), microbuilder:RESISTOR2512
- added R3+, R3-: (no value), wirepad:1,6/0,9
- added R4: 10K, microbuilder:RESISTOR_4PACK
- JP3: device microbuilder:HEADER-1X16_76MIL -> microbuilder:HEADER-1X2ROUND
Connections:
- removed net A: JP3.12, MS1.GPIOA0
- removed net AREF: JP3.14, MS1.AREF
- removed net B: JP3.11, MS1.GPIOA1
- removed net C: JP3.10, MS1.GPIOA2
- removed net D: JP3.9, MS1.GPIOA3
- removed net E: JP3.8, MS1.GPIOA4
- removed net EN: JP1.2, MS1.EN
- removed net F: JP3.7, MS1.GPIOA5
- removed net G: JP3.1, MS1.NC
- removed net H: JP1.10, MS1.GPIO5
- removed net I: JP1.9, MS1.GPIO6
- removed net J: JP1.8, MS1.GPIO9
- removed net K: JP1.7, MS1.GPIO10
- removed net L: JP1.6, MS1.GPIO11
- removed net M: JP1.5, MS1.GPIO12
- removed net MISO: JP3.4, MS1.GPIOMISO
- removed net MOSI: JP3.5, MS1.GPIOMOSI
- removed net N: JP1.4, MS1.GPIO13
- removed net RESET: JP3.16, MS1.!RESET
- removed net RX: JP3.3, MS1.GPIORX
- removed net SCK: JP3.6, MS1.GPIOSCK
- removed net TX: JP3.2, MS1.GPIOTX
- removed net USB: JP1.3, MS1.USB
- removed net VBAT: JP1.1, MS1.VBAT
- net 3.3V: now also R4G$3.2, R4G$4.2; no longer JP3.15, R6G$3.2, R6G$4.2
- net GND: now also R4G$1.2, R4G$2.2; no longer JP3.13, R6G$1.2, R6G$2.2
- net N$1: now also R2G$1.1; no longer R6G$1.1
- net N$2: now also R2G$2.1; no longer R6G$2.1
- net N$3: now also R4G$1.1; no longer R2G$1.1
- net N$4: now also R4G$2.1; no longer R2G$2.1
- net SCL: now also R4G$3.1; no longer JP1.11, R6G$3.1
- net SDA: now also R4G$4.1; no longer JP1.12, R6G$4.1
- net VIN1+: now also JP3.2, R1+.P, R1.2; no longer JP2.2, R5+.P, R5.2
- net VIN1-: now also JP3.1, R1-.P, R1.1; no longer JP2.1, R5-.P, R5.1
- net VIN2+: now also R3+.P, R3.2; no longer R1+.P, R1.2
- net VIN2-: now also R3-.P, R3.1; no longer R1-.P, R1.1
Other:
- moved on the sheet: R1, R1+, R1-, R2G$1, R2G$2, R2G$3, R2G$4
