File: Adafruit/INA219x4 DoubleWing.brd (EAGLE design)
At the start: 50.8 x 47 mm, 42 parts, among them J1 5mm, J2 5mm, J3 5mm, J4 5mm, U1 INA219BIDCNT, U2 INA219BIDCNT, U3 INA219BIDCNT, U4 INA219BIDCNT

Commit message: Updated to version that was sent to oshpark for fabrication
Parts:
- removed JP1, JP2, JP3, JP4: (no value), microbuilder:1X02_ROUND
- added J5, J7: 5mm, SparkFun-Connectors:SCREWTERMINAL-5MM-2
- added J6, J8: (no value), SparkFun-Connectors:1X01
- J2, J4: value 5mm -> (none); device SparkFun-Connectors:SCREWTERMINAL-5MM-2 -> SparkFun-Connectors:1X01
- moved J3 53.7 mm to (3.81, 7.49), turned to 90 degrees
- moved J2 43.2 mm to (47.0, 5.33), turned to 0 degrees
- moved J4 14.3 mm to (4.70, 17.4), turned to 0 degrees
Connections:
- net GND: now also J2.1, J4.1, J6.1, J8.1
- net VIN1+: no longer JP1.2
- net VIN1-: no longer JP1.1
- net VIN2+: now also J3.2; no longer J2.2, JP2.2
- net VIN2-: now also J3.1; no longer J2.1, JP2.1
- net VIN3+: now also J5.2; no longer J3.2, JP3.2
- net VIN3-: now also J5.1; no longer J3.1, JP3.1
- net VIN4+: now also J7.2; no longer J4.2, JP4.2
- net VIN4-: now also J7.1; no longer J4.1, JP4.1
Routing:
- net GND: track 150.6 -> 187.1 mm, vias 16 -> 18
- net VIN4-: track 23.9 -> 13.2 mm
- net VIN3-: track 23.4 -> 12.8 mm
- net VIN2-: track 23.5 -> 13.0 mm
- net VIN1-: track 23.5 -> 13.0 mm
- net VIN4+: track 18.2 -> 13.5 mm
- net VIN3+: track 18.0 -> 13.5 mm
- net VIN1+: track 17.7 -> 13.3 mm
- net VIN2+: track 17.7 -> 13.3 mm
- net N$18: track 25.1 -> 24.1 mm
- net SDA: track 128.1 -> 127.1 mm
Other:
- board text added: "+26V ±3.2A"
- board text added: "DoubleWing INA219x4 v1 +26V ±3.2A"
