File: Adafruit/INA219x4_DoubleWing.sch (EAGLE design)
At the start: 42 parts, among them J1 5mm, J3 5mm, J5 5mm, J7 5mm, U1 INA219BIDCNT, U2 INA219BIDCNT, U3 INA219BIDCNT, U4 INA219BIDCNT

Commit message: INA219x4 DoubleWing v2.0
Parts:
- removed A0, A1, A2, A3, A4, A5, A6, A7: (no value), microbuilder:SOLDERJUMPERREFLOW_NOPASTE
- removed J1, J3, J5, J7: 5mm, SparkFun-Connectors:CONN_025MM
- removed J2, J4, J6, J8: (no value), SparkFun-Connectors:CONN_01
- removed R1, R3, R5, R7: 0.1/1% (PT2512FK-070R1L), microbuilder:RESISTOR2512
- removed R1+, R1-, R3+, R3-, R5+, R5-, R7+, R7-: (no value), wirepad:1,6/0,9
- removed R2, R4, R6, R8: 10K, microbuilder:RESISTOR_4PACK
- added J1#1, J1#2, J1#3, J1#4: 5mm, SparkFun-Connectors:CONN_025MM
- added J2#1, J2#2, J2#3, J2#4: (no value), SparkFun-Connectors:CONN_01
- added JMPA0.1#1, JMPA0.1#2, JMPA0.1#3, JMPA0.1#4, JMPA0.2#1, JMPA0.2#2, JMPA0.2#3, JMPA0.2#4, JMPA1.1#1, JMPA1.1#2, JMPA1.1#3, JMPA1.1#4, JMPA1.2#1, JMPA1.2#2, JMPA1.2#3, JMPA1.2#4: 0R-JUMPD, pv_jump-0r-smd:0R-JUMPD
- added R1#1, R1#2, R1#3, R1#4: 0.1/1% (PT2512FK-070R1L), microbuilder:RESISTOR2512
- added R1+#1, R1+#2, R1+#3, R1+#4, R1-#1, R1-#2, R1-#3, R1-#4: (no value), wirepad:1,6/0,9
- added R2#1, R2#2, R2#3, R2#4: 10K, microbuilder:RESISTOR_4PACK
Connections:
- removed net N$16: A1.2, R2G$1.1, U1.A1
- removed net N$24: A5.2, R6G$1.1, U3.A1
- removed net N$25: A4.2, R6G$2.1, U3.A0
- removed net N$26: A0.2, R2G$2.1, U1.A0
- removed net N$27: A3.2, R4G$1.1, U2.A1
- removed net N$28: A2.2, R4G$2.1, U2.A0
- removed net N$29: A7.2, R8G$1.1, U4.A1
- removed net N$30: A6.2, R8G$2.1, U4.A0
- new net A0#1: JMPA0.1#1-0R.2, JMPA0.2#1-0R.2, R2#1G$2.1, U1.A0
- new net A0#2: JMPA0.1#2-0R.2, JMPA0.2#2-0R.2, R2#2G$2.1, U2.A0
- new net A0#3: JMPA0.1#3-0R.2, JMPA0.2#3-0R.2, R2#3G$2.1, U3.A0
- new net A0#4: JMPA0.1#4-0R.2, JMPA0.2#4-0R.2, R2#4G$2.1, U4.A0
- new net A1#1: JMPA1.1#1-0R.2, JMPA1.2#1-0R.2, R2#1G$1.1, U1.A1
- new net A1#2: JMPA1.1#2-0R.2, JMPA1.2#2-0R.2, R2#2G$1.1, U2.A1
- new net A1#3: JMPA1.1#3-0R.2, JMPA1.2#3-0R.2, R2#3G$1.1, U3.A1
- new net A1#4: JMPA1.1#4-0R.2, JMPA1.2#4-0R.2, R2#4G$1.1, U4.A1
- net 3.3V: now also JMPA0.1#1-0R.1, JMPA0.1#2-0R.1, JMPA0.1#3-0R.1, JMPA0.1#4-0R.1, JMPA1.1#1-0R.1, JMPA1.1#2-0R.1, JMPA1.1#3-0R.1, JMPA1.1#4-0R.1, R2#1G$3.2, R2#1G$4.2, R2#2G$3.2, R2#2G$4.2, R2#3G$3.2, R2#3G$4.2, R2#4G$3.2, R2#4G$4.2; no longer A0.1, A1.1, A2.1, A3.1, A4.1, A5.1, A6.1, A7.1, R2G$3.2, R2G$4.2, R4G$3.2, R4G$4.2, R6G$3.2, R6G$4.2, R8G$3.2, R8G$4.2
- net GND: now also J2#1.1, J2#2.1, J2#3.1, J2#4.1, JMPA0.2#1-0R.3, JMPA0.2#2-0R.3, JMPA0.2#3-0R.3, JMPA0.2#4-0R.3, JMPA1.2#1-0R.3, JMPA1.2#2-0R.3, JMPA1.2#3-0R.3, JMPA1.2#4-0R.3, R2#1G$1.2, R2#1G$2.2, R2#2G$1.2, R2#2G$2.2, R2#3G$1.2, R2#3G$2.2, R2#4G$1.2, R2#4G$2.2; no longer J2.1, J4.1, J6.1, J8.1, R2G$1.2, R2G$2.2, R4G$1.2, R4G$2.2, R6G$1.2, R6G$2.2, R8G$1.2, R8G$2.2
- net SCL: now also JMPA0.1#1-0R.3, JMPA0.1#2-0R.3, JMPA0.1#3-0R.3, JMPA0.1#4-0R.3, JMPA1.1#1-0R.3, JMPA1.1#2-0R.3, JMPA1.1#3-0R.3, JMPA1.1#4-0R.3, R2#1G$4.1, R2#2G$4.1, R2#3G$4.1, R2#4G$4.1; no longer R2G$3.1, R4G$3.1, R6G$3.1, R8G$3.1
- net SDA: now also JMPA0.2#1-0R.1, JMPA0.2#2-0R.1, JMPA0.2#3-0R.1, JMPA0.2#4-0R.1, JMPA1.2#1-0R.1, JMPA1.2#2-0R.1, JMPA1.2#3-0R.1, JMPA1.2#4-0R.1, R2#1G$3.1, R2#2G$3.1, R2#3G$3.1, R2#4G$3.1; no longer R2G$4.1, R4G$4.1, R6G$4.1, R8G$4.1
- net VIN1+: now also J1#1.2, R1#1.2, R1+#1.P; no longer J1.2, R1+.P, R1.2
- net VIN1-: now also J1#1.1, R1#1.1, R1-#1.P; no longer J1.1, R1-.P, R1.1
- net VIN2+: now also J1#2.2, R1#2.2, R1+#2.P; no longer J3.2, R3+.P, R3.2
- net VIN2-: now also J1#2.1, R1#2.1, R1-#2.P; no longer J3.1, R3-.P, R3.1
- net VIN3+: now also J1#3.2, R1#3.2, R1+#3.P; no longer J5.2, R5+.P, R5.2
- net VIN3-: now also J1#3.1, R1#3.1, R1-#3.P; no longer J5.1, R5-.P, R5.1
- net VIN4+: now also J1#4.2, R1#4.2, R1+#4.P; no longer J7.2, R7+.P, R7.2
- net VIN4-: now also J1#4.1, R1#4.1, R1-#4.P; no longer J7.1, R7-.P, R7.1
Other:
- moved on the sheet: C1, C2, C3, C4, U1, U2, U3, U4
